File: KiCad Test Board/Board v2.0/Board.kicad_pcb (KiCad board)
At the start: 2 copper layers, 95.2 x 88.9 mm, 28 parts, among them J1 Conn_01x11, J2 Screw_Terminal_01x04, U1 ADG732BSUZ

Commit message: Updated KiCad project files
Parts:
- R2: value 1M -> 1k; footprint Resistor_SMD:R_2512_6332Metric_Pad1.52x3.35mm_HandSolder -> Resistor_SMD:R_MiniMELF_MMA-0204
- moved R2 1.11 mm to (52.2, 79.1)
Routing:
- net GND: vias 51 -> 49
Changed lines of the file:
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@@
   )
   (setup
-    (last_trace_width 0.127)
+    (last_trace_width 0.635)
     (user_trace_width 0.254)
     (user_trace_width 0.635)
@@
     )
   )
-  (module Resistor_SMD:R_2512_6332Metric_Pad1.52x3.35mm_HandSolder (layer F.Cu)
-    (at 51.1145 79.121 180)
-    (descr "Resistor SMD 2512 (6332 Metric), square (rectangular) end terminal, IPC_7351 nominal with elongated pad for handsoldering. (Body size source: http://www.tortai-tech.com/upload/download/2011102023233369053.pdf), generated with kicad-footprint-generator")
-    (tags "resistor handsolder")
-    (attr smd)
-    (fp_text reference R2 (at 5.2675 0) (layer F.SilkS)
-      (effects (font (size 1 1) (thickness 0.15)))
-    )
-    (fp_text value 1M (at 0 2.62) (layer F.Fab)
-      (effects (font (size 1 1) (thickness 0.15)))
-    )
-    (fp_text user %R (at 0 0) (layer F.Fab)
-      (effects (font (size 1 1) (thickness 0.15)))
-    )
-    (fp_line (start 4 1.92) (end -4 1.92) (layer F.CrtYd) (width 0.05))
-    (fp_line (start 4 -1.92) (end 4 1.92) (layer F.CrtYd) (width 0.05))
-    (fp_line (start -4 -1.92) (end 4 -1.92) (layer F.CrtYd) (width 0.05))
-    (fp_line (start -4 1.92) (end -4 -1.92) (layer F.CrtYd) (width 0.05))
-    (fp_line (start -2.052064 1.71) (end 2.052064 1.71) (layer F.SilkS) (width 0.12))
-    (fp_line (start -2.052064 -1.71) (end 2.052064 -1.71) (layer F.SilkS) (width 0.12))
-    (fp_line (start 3.15 1.6) (end -3.15 1.6) (layer F.Fab) (width 0.1))
-    (fp_line (start 3.15 -1.6) (end 3.15 1.6) (layer F.Fab) (width 0.1))
-    (fp_line (start -3.15 -1.6) (end 3.15 -1.6) (layer F.Fab) (width 0.1))
-    (fp_line (start -3.15 1.6) (end -3.15 -1.6) (layer F.Fab) (width 0.1))
-    (pad 2 smd roundrect (at 2.9875 0 180) (size 1.525 3.35) (layers F.Cu F.Paste F.Mask) (roundrect_rratio 0.163934)
-      (net 36 LCR_HIGH1))
-    (pad 1 smd roundrect (at -2.9875 0 180) (size 1.525 3.35) (layers F.Cu F.Paste F.Mask) (roundrect_rratio 0.163934)
-      (net 20 "Net-(R2-Pad1)"))
-    (model ${KISYS3DMOD}/Resistor_SMD.3dshapes/R_2512_6332Metric.wrl
-      (at (xyz 0 0 0))
-      (scale (xyz 1 1 1))
-      (rotate (xyz 0 0 0))
-    )
-    (model "/Users/CollinHeist/Documents/Academia/AgMEQ Lab/KiCad Libraries/kicad-packages3D-5.1.4/Resistor_SMD.3dshapes/R_2512_6332Metric.step"
-      (at (xyz 0 0 0))
-      (scale (xyz 1 1 1))
-      (rotate (xyz 0 0 0))
-    )
-  )
   (module Resistor_SMD:R_1206_3216Metric_Pad1.42x1.75mm_HandSolder (layer F.Cu)
     (at 52.7415 75.565 180)
@@
     )
   )
+  (module Resistor_SMD:R_MiniMELF_MMA-0204 (layer F.Cu)
+    (at 52.221 79.121 180)
+    (descr "Resistor, MiniMELF, MMA-0204, http://www.vishay.com/docs/28713/melfprof.pdf")
+    (tags "MiniMELF Resistor")
+    (attr smd)
+    (fp_text reference R2 (at 3.58 0) (layer F.SilkS)
+      (effects (font (size 1 1) (thickness 0.15)))
+    )
+    (fp_text value 1k (at 0 1.7) (layer F.Fab)
+      (effects (font (size 1 1) (thickness 0.15)))
+    )
+    (fp_text user %R (at 0 0) (layer F.Fab)
+      (effects (font (size 0.6 0.6) (thickness 0.12)))
+    )
+    (fp_line (start 0.6 0.85) (end -0.6 0.85) (layer F.SilkS) (width 0.12))
+    (fp_line (start -0.6 -0.85) (end 0.6 -0.85) (layer F.SilkS) (width 0.12))
+    (fp_line (start 0.9 0.7) (end 0.9 -0.7) (layer F.Fab) (width 0.12))
+    (fp_line (start -0.9 -0.7) (end -0.9 0.7) (layer F.Fab) (width 0.12))
+    (fp_line (start -1.8 -0.7) (end -1.8 0.7) (layer F.Fab) (width 0.12))
+    (fp_line (start -1.8 0.7) (end 1.8 0.7) (layer F.Fab) (width 0.12))
+    (fp_line (start 1.8 0.7) (end 1.8 -0.7) (layer F.Fab) (width 0.12))
+    (fp_line (start 1.8 -0.7) (end -1.8 -0.7) (layer F.Fab) (width 0.12))
+    (fp_line (start -2.5 -1.15) (end 2.5 -1.15) (layer F.CrtYd) (width 0.05))
+    (fp_line (start -2.5 -1.15) (end -2.5 1.15) (layer F.CrtYd) (width 0.05))
+    (fp_line (start 2.5 1.15) (end 2.5 -1.15) (layer F.CrtYd) (width 0.05))
+    (fp_line (start 2.5 1.15) (end -2.5 1.15) (layer F.CrtYd) (width 0.05))
+    (pad 1 smd rect (at -1.5 0 180) (size 1.5 1.8) (layers F.Cu F.Paste F.Mask)
+      (net 20 "Net-(R2-Pad1)"))
+    (pad 2 smd rect (at 1.5 0 180) (size 1.5 1.8) (layers F.Cu F.Paste F.Mask)
+      (net 36 LCR_HIGH1))
+    (model ${KISYS3DMOD}/Resistor_SMD.3dshapes/R_MiniMELF_MMA-0204.wrl
+      (at (xyz 0 0 0))
+      (scale (xyz 1 1 1))
+      (rotate (xyz 0 0 0))
+    )
+  )
   (gr_text "LCR\nHIGH2" (at 76.708 38.862 270) (layer F.SilkS)
     (effects (font (size 0.635 0.635) (thickness 0.1016)) (justify left))
@@
   (via (at 38.1 38.1) (size 0.4572) (drill 0.254) (layers F.Cu B.Cu) (net 1))
   (via (at 38.1 50.8) (size 0.4572) (drill 0.254) (layers F.Cu B.Cu) (net 1))
-  (via (at 40.386 43.434) (size 0.4572) (drill 0.254) (layers F.Cu B.Cu) (net 1))
-  (via (at 40.386 56.134) (size 0.4572) (drill 0.254) (layers F.Cu B.Cu) (net 1))
-  (via (at 40.386 68.834) (size 0.4572) (drill 0.254) (layers F.Cu B.Cu) (net 1))
   (via (at 38.1 101.6) (size 0.4572) (drill 0.254) (layers F.Cu B.Cu) (net 1))
   (via (at 50.8 101.6) (size 0.4572) (drill 0.254) (layers F.Cu B.Cu) (net 1))
@@
   (via (at 76.2 101.6) (size 0.4572) (drill 0.254) (layers F.Cu B.Cu) (net 1))
   (via (at 88.9 101.6) (size 0.4572) (drill 0.254) (layers F.Cu B.Cu) (net 1))
-  (via (at 39.243 55.372) (size 0.4572) (drill 0.254) (layers F.Cu B.Cu) (net 1))
   (via (at 50.8 38.1) (size 0.4572) (drill 0.254) (layers F.Cu B.Cu) (net 1))
   (via (at 63.5 38.1) (size 0.4572) (drill 0.254) (layers F.Cu B.Cu) (net 1))
@@
   (via (at 44.45 69.85) (size 0.4572) (drill 0.254) (layers F.Cu B.Cu) (net 1))
   (via (at 44.45 82.55) (size 0.4572) (drill 0.254) (layers F.Cu B.Cu) (net 1))
-  (via (at 39.243 42.672) (size 0.4572) (drill 0.254) (layers F.Cu B.Cu) (net 1))
   (via (at 95.25 82.55) (size 0.4572) (drill 0.254) (layers F.Cu B.Cu) (net 1))
   (segment (start 65.436001 66.771001) (end 65.936001 66.771001) (width 0.254) (layer F.Cu) (net 1))
@@
   (segment (start 74.549 93.218) (end 74.549 94.420081) (width 1.27) (layer F.Cu) (net 1))
   (segment (start 74.549 94.420081) (end 74.549 95.6056) (width 1.27) (layer F.Cu) (net 1))
+  (via (at 38.1 63.5) (size 0.4572) (drill 0.254) (layers F.Cu B.Cu) (net 1))
+  (via (at 38.1 76.2) (size 0.4572) (drill 0.254) (layers F.Cu B.Cu) (net 1))
+  (via (at 38.1 88.9) (size 0.4572) (drill 0.254) (layers F.Cu B.Cu) (net 1))
   (segment (start 66.936001 85.590999) (end 66.936001 75.111001) (width 0.254) (layer F.Cu) (net 2))
   (segment (start 59.309 93.218) (end 66.936001 85.590999) (width 0.254) (layer F.Cu) (net 2))
@@
   (segment (start 63.016001 74.524999) (end 54.102 83.439) (width 0.254) (layer F.Cu) (net 19))
   (segment (start 63.016001 73.691001) (end 63.016001 74.524999) (width 0.254) (layer F.Cu) (net 19))
-  (segment (start 60.031999 73.191001) (end 54.102 79.121) (width 0.254) (layer F.Cu) (net 20))
-  (segment (start 63.016001 73.191001) (end 60.031999 73.191001) (width 0.254) (layer F.Cu) (net 20))
+  (segment (start 53.721 78.971) (end 53.721 79.121) (width 0.254) (layer F.Cu) (net 20))
+  (segment (start 59.500999 73.191001) (end 53.721 78.971) (width 0.254) (layer F.Cu) (net 20))
+  (segment (start 63.016001 73.191001) (end 59.500999 73.191001) (width 0.254) (layer F.Cu) (net 20))
   (segment (start 57.102999 72.691001) (end 54.229 75.565) (width 0.254) (layer F.Cu) (net 21))
   (segment (start 63.016001 72.691001) (end 57.102999 72.691001) (width 0.254) (layer F.Cu) (net 21))
@@
   (segment (start 67.936001 92.210999) (end 67.936001 75.111001) (width 0.254) (layer F.Cu) (net 35))
   (segment (start 66.929 93.218) (end 67.936001 92.210999) (width 0.254) (layer F.Cu) (net 35))
-  (segment (start 48.127 83.439) (end 48.127 79.121) (width 0.635) (layer F.Cu) (net 36))
-  (segment (start 48.127 79.121) (end 48.127 78.692) (width 0.635) (layer F.Cu) (net 36))
   (segment (start 82.169 49.911) (end 84.709 52.451) (width 0.635) (layer F.Cu) (net 36))
   (segment (start 84.709 63.808) (end 84.636 63.881) (width 0.635) (layer F.Cu) (net 36))
@@
   (segment (start 51.254 75.565) (end 51.254 55.318) (width 0.635) (layer F.Cu) (net 36))
   (segment (start 51.254 55.318) (end 51.181 55.245) (width 0.635) (layer F.Cu) (net 36))
-  (segment (start 48.127 78.692) (end 51.254 75.565) (width 0.635) (layer F.Cu) (net 36))
   (segment (start 51.181 55.245) (end 56.515 49.911) (width 0.635) (layer F.Cu) (net 36))
   (segment (start 75.438 49.911) (end 82.169 49.911) (width 0.635) (layer F.Cu) (net 36))
@@
   (segment (start 76.652 46.284) (end 73.206 49.73) (width 0.635) (layer F.Cu) (net 36))
   (segment (start 76.652 34.544) (end 76.652 46.284) (width 0.635) (layer F.Cu) (net 36))
+  (segment (start 51.254 78.588) (end 50.721 79.121) (width 0.635) (layer F.Cu) (net 36))
+  (segment (start 51.254 75.565) (end 51.254 78.588) (width 0.635) (layer F.Cu) (net 36))
+  (segment (start 50.721 80.845) (end 48.127 83.439) (width 0.635) (layer F.Cu) (net 36))
+  (segment (start 50.721 79.121) (end 50.721 80.845) (width 0.635) (layer F.Cu) (net 36))
   (via (at 67.056 63.246) (size 0.4572) (drill 0.254) (layers F.Cu B.Cu) (net 37))
   (segment (start 66.936001 65.772001) (end 66.936001 66.771001) (width 0.254) (layer F.Cu) (net 37))
