File: Board Redesign/KiCad Project/Team-FIRE-v2/schematic-2.sch (KiCad schematic (older format))
At the start: 14 parts

Commit message: Added I2C Expander
- Added all required connections for the I2C expander
Parts:
- added C? (x2): 0.1uF, Capacitor_SMD:C_0603_1608Metric, symbol Device:C
- added R? (x2): 10k, Resistor_SMD:R_0603_1608Metric, symbol Device:R
Connections:
- net labels added: 3959_EN,3.6C, 3959_GOOD,3.6C, 5V_EN,3.1A, 8V_EN,3.1B, BOOST_EN,3.5C, EN_TES_BUS,3.5D, I2C_LED, PWR_EN,3.4E, PWR_SW,3.3D, SCL,3.6D, SDA,3.6D, TX_ACTIVE,3.5C
- wire segments 85 -> 128
- no-connect marks 0 -> 6
Other:
- note added: "I2C Translators\n"

Commit message: Made more progress on board redesign
- Primarily deleted useless (for our purposes) items from the old schematic so we do not have to spend time transferring them over.
- Finished some component transfer
- Renamed some folders
Parts:
- removed C? (x2): 0.1uF, Capacitor_SMD:C_0603_1608Metric, symbol Device:C
- removed R?: 10k, Resistor_SMD:R_0603_1608Metric, symbol Device:R
- removed U?: TXB0108DQSR, Package_SON:USON-20_2x4mm_P0.4mm, symbol Logic_LevelTranslator:TXB0108DQSR
- added C?: 0.1uF, Capacitor_SMD:C_0603_1608Metric, symbol Device:C
Connections:
- net labels added: 3.3V_SENSE, 3959_EN, 3959_GOOD, 5V_EN, 8V_EN, BOOST_EN, CTS, DCD, DSR, DTR, EN_IR_BUS, EN_TES_BUS, PWR_EN, PWR_SW, RI, RTS, RX, SCL, SDA, TES-GPS-FLAG, TES-RX, TES-SPARE, TES-TX, TX, TX_ACTIVE
- net labels removed: 3.3V_SENSE,3.5C, 3959_EN,3.6C, 3959_GOOD,3.6C, 5V_EN,3.1A, 8V_EN,3.1B, BOOST_EN,3.5C, CTS,1.5B, DCD,1.6B, DSR,1.5B, DTR,1.6B, EN_IR_BUS,3.5D, EN_TES_BUS,3.5D, I2C_LED, PWR_EN,3.4E, PWR_SW,3.3D, RI,1.6B, RS232-CDC,3.1E, RS232-CRS,3.1E, RS232-DSR,3.1E, RS232-DTR,3.1E, RS232-RI,3.1E, RS232-RTS,3.1E, RS232-RX,3.1E, RTS,1.5B, RX,1.5B, SCL,3.6D, SDA,3.6D, TX,1.6B, TX_ACTIVE,1.5B, TX_ACTIVE,3.5C
- wire segments 128 -> 99
- no-connect marks 6 -> 7
Other:
- note added: "I2C Expander"
- note added: "VCCB is typically\ntied to 3.3V"
- note removed: "I2C Translators\n"
- moved on the sheet: C?, J?, R?, U?

Commit message: Added Shelby's work
Parts:
- added D? (x2): Blue, symbol Device:LED_Small
- added D? (x2): Orange, symbol Device:LED_Small
- added J?: Conn_ARM_JTAG_SWD_10, symbol Connector:Conn_ARM_JTAG_SWD_10
- added J?: USB_B_Mini, symbol Connector:USB_B_Mini
- added R? (x4): 330, Resistor_SMD:R_0603_1608Metric, symbol Device:R
- gave numbers to parts that had none: 1
Connections:
- net labels added: I2_LED, RST, RX_LED, SWCLK, SWDIO, SYS_LED, TX_LED, USB_D+, USB_D-
- wire segments 99 -> 131
Other:
- note added: "Keep reset button?"
- note added: "SAMD...21 or 51"
- note added: "uC Support"

Commit message: Added SAMD51
- Created schematic symbol, footprint, and 3D model for the SAMD51
- Added SAMD51 to the schematic (only partially implemented)
- Added decoupling capacitors to the 3.3V bus (as recommended by the SAMD51 design manual)
- Started checklist for SAMD51 implementation on the top-level schematic sheet; there's no convenient breakout board to emulate
- Implemented power connections for SAMD51
Parts:
- removed C? (x2): 0.1uF, Capacitor_SMD:C_0603_1608Metric, symbol Device:C
- removed IC?: SX1509BIULTRT, QFN40P400X400X60-29N-D, symbol Team-FIRE:SX1509BIULTRT
- removed R? (x2): 10k, Resistor_SMD:R_0603_1608Metric, symbol Device:R
- added C?: 4.7uF, Capacitor_SMD:C_0603_1608Metric, symbol Device:C
- added C? (x7): 100nF, Capacitor_SMD:C_0603_1608Metric, symbol Device:C
- added IC? (x2): SAMD51, Package_QFP:TQFP-100_14x14mm_P0.5mm, symbol Team-FIRE:SAMD51
- added L?: 10uH, Inductor_SMD:L_0603_1608Metric, symbol Device:L
Connections:
- net labels removed: 3959_EN, 3959_GOOD, 5V_EN, 8V_EN, BOOST_EN, EN_TES_BUS, PWR_EN, PWR_SW, SCL, SDA
- wire segments 131 -> 149
- no-connect marks 7 -> 0
Other:
- note added: "Pin 12"
- note added: "Pin 39"
- note added: "Pin 51"
- note added: "Pin 63"
- note added: "Pin 77"
- note added: "Pin 89\n"
- note added: "Pin 91\n"
- note added: "Pin 92"
- note added: "Place all components near\ntheir respective pins.\nChoose low ESR capacitors."
- note removed: "I2C Expander"
- moved on the sheet: D?, J?, R?

Commit message: Smol changes
Other:
- note added: "SAMD 51"
- note removed: "SAMD...21 or 51"
Changed lines of the file:
@@
 EESchema Schematic File Version 4
-LIBS:Team-FIRE-v2-cache
 EELAYER 30 0
 EELAYER END
@@
 VCCB is typically\ntied to 3.3V
 Text Notes 8200 700  0    79   ~ 16
-SAMD...21 or 51
+SAMD 51
 Wire Notes Line
 	6400 7550 6400 5750
