File: Board Redesign/KiCad Project/Team-FIRE-v2/schematic-2.sch (KiCad schematic (older format))
At the start: 39 parts, among them IC1 SAMD51, J3 USB_B_Mini, J4 Conn_01x03, J5 Conn_ARM_JTAG_SWD_10, SW1 RESET, U4 TXB0108DQSR, U5 ATSAMD51N20A-AU, U7 TXB0104RUT, Y1 32.768kHz

Commit message: Progress
- Corrected many footprint errors on components
- Finalized work on schematic 3
Parts:
- C21: footprint (none) -> Capacitor_SMD:C_0603_1608Metric
- J5: footprint (none) -> Connector_PinHeader_1.27mm:PinHeader_2x05_P1.27mm_Vertical_SMD; MPN (none) -> FTSH-105-01-L-DV-K-TR
- JP2: footprint (none) -> Jumper:SolderJumper-3_P1.3mm_Bridged2Bar12_RoundedPad1.0x1.5mm
- R12, R14, R17: footprint (none) -> Resistor_SMD:R_0603_1608Metric
Changed lines of the file:
@@
 F 0 "J5" V 2369 6750 50  0000 C CNN
 F 1 "Conn_ARM_JTAG_SWD_10" V 2460 6750 50  0000 C CNN
-F 2 "" H 2950 6750 50  0001 C CNN
+F 2 "Connector_PinHeader_1.27mm:PinHeader_2x05_P1.27mm_Vertical_SMD" H 2950 6750 50  0001 C CNN
 F 3 "http://infocenter.arm.com/help/topic/com.arm.doc.ddi0314h/DDI0314H_coresight_components_trm.pdf" V 2600 5500 50  0001 C CNN
+F 4 "FTSH-105-01-L-DV-K-TR" V 2950 6750 50  0001 C CNN "MPN"
 	1    2950 6750
 	0    1    1    0
@@
 F 0 "R14" H 5170 4846 50  0000 L CNN
 F 1 "10k" H 5170 4755 50  0000 L CNN
-F 2 "" V 5030 4800 50  0001 C CNN
+F 2 "Resistor_SMD:R_0603_1608Metric" V 5030 4800 50  0001 C CNN
 F 3 "~" H 5100 4800 50  0001 C CNN
 	1    5100 4800
@@
 F 0 "R12" V 4643 5050 50  0000 C CNN
 F 1 "330" V 4734 5050 50  0000 C CNN
-F 2 "" V 4780 5050 50  0001 C CNN
+F 2 "Resistor_SMD:R_0603_1608Metric" V 4780 5050 50  0001 C CNN
 F 3 "~" H 4850 5050 50  0001 C CNN
 	1    4850 5050
@@
 F 0 "C21" H 5215 5346 50  0000 L CNN
 F 1 "100nF" H 5215 5255 50  0000 L CNN
-F 2 "" H 5100 5300 50  0001 C CNN
+F 2 "Capacitor_SMD:C_0603_1608Metric" H 5100 5300 50  0001 C CNN
 F 3 "~" H 5100 5300 50  0001 C CNN
 	1    5100 5300
@@
 F 0 "R17" H 6570 4646 50  0000 L CNN
 F 1 "1k" H 6570 4555 50  0000 L CNN
-F 2 "" V 6430 4600 50  0001 C CNN
+F 2 "Resistor_SMD:R_0603_1608Metric" V 6430 4600 50  0001 C CNN
 F 3 "~" H 6500 4600 50  0001 C CNN
 	1    6500 4600
@@
 F 0 "JP2" H 1400 1213 50  0000 C CNN
 F 1 "SolderJumper_3_Bridged12" H 1400 1214 50  0001 C CNN
-F 2 "" H 1400 1100 50  0001 C CNN
+F 2 "Jumper:SolderJumper-3_P1.3mm_Bridged2Bar12_RoundedPad1.0x1.5mm" H 1400 1100 50  0001 C CNN
 F 3 "~" H 1400 1100 50  0001 C CNN
 	1    1400 1100
