File: Board Redesign/KiCad Project/Team-FIRE-v2/schematic-2.sch (KiCad schematic (older format))
At the start: 39 parts, among them U7 TXB0104RUT

Commit message: Fix: updated some comments
Other:
- note added: "SAMD51 Checklist:\n- From https://www.mouser.com/datasheet/2/268/60001507E-1660031.pdf#page=2096&zoom=100,0,0\n- Voltage of [1.71, 3.63] V must be applied to VDDIO and VDDANA.\n- Voltage VDDIOB must be lower or equal to VDDIO / VDDANA.\n- Verify the power supply is appropriately set for Switching / Linear mode.\n+ We need a pull-up resistor on the SWCLK pin\n+ We need a RC filter on ~RESET\n- We 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"
- note added: "The SAMD51 symbol:\n- should be updated to include pin types (input/output, etc)\n- should be divided into more (functional) units. \nRight now it is taking too much space"
- note added: "We might need to put the decoupling capacitors into the uC support block"
- note removed: "SAMD51 Checklist:\n- From https://www.mouser.com/datasheet/2/268/60001507E-1660031.pdf#page=2096&zoom=100,0,0\n- Voltage of [1.71, 3.63] V must be applied to VDDIO and VDDANA.\n- Voltage VDDIOB must be lower or equal to VDDIO / VDDANA.\n- Verify the power supply is appropriately set for Switching / Linear mode.\n- We need a pull-up resistor on the SWCLK pin\n- We need a RC filter on ~RESET\n- We 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"
- note removed: "The SAMD51 symbol:\n- should be updated to include pin types (input/output, etc)\n- should be divided into (functional) units. Right now it is taking too much space"
- note removed: "We might need to put the decoupling capacitors into the uC support block\nAlso, there are two more decoupling capacitors on sheet 1/3, so technically \ntwo mores capacitor are added to this list. Maybe we should remove the one \none sheet 1/3 and keep these ones below?"
Changed lines of the file:
@@
 	8700 1850 10300 1850
 Text Notes 6950 6300 0    50   ~ 0
-SAMD51 Checklist:\n- From https://www.mouser.com/datasheet/2/268/60001507E-1660031.pdf#page=2096&zoom=100,0,0\n- Voltage of [1.71, 3.63] V must be applied to VDDIO and VDDANA.\n- Voltage VDDIOB must be lower or equal to VDDIO / VDDANA.\n- Verify the power supply is appropriately set for Switching / Linear mode.\n- We need a pull-up resistor on the SWCLK pin\n- We need a RC filter on ~RESET\n-  We need to eliminate or attenuate noise in\norder to avoid that it reaches supply pins, I/O pins and crystals.
+SAMD51 Checklist:\n- From https://www.mouser.com/datasheet/2/268/60001507E-1660031.pdf#page=2096&zoom=100,0,0\n- Voltage of [1.71, 3.63] V must be applied to VDDIO and VDDANA.\n- Voltage VDDIOB must be lower or equal to VDDIO / VDDANA.\n- Verify the power supply is appropriately set for Switching / Linear mode.\n+ We need a pull-up resistor on the SWCLK pin\n+ We need a RC filter on ~RESET\n-  We need to eliminate or attenuate noise in\norder to avoid that it reaches supply pins, I/O pins and crystals.
 $Comp
 L power:+3.3V #PWR?
@@
 Text Notes 4050 4250 0    40   ~ 0
 A software reset is nice. But, we might need to\n manually reset the SAMD.
-Text Notes 7250 3900 0    50   ~ 0
-The SAMD51 symbol:\n- should be updated to include pin types (input/output, etc)\n- should be divided into (functional) units. Right now it is taking too much space
+Text Notes 7350 3950 0    50   ~ 0
+The SAMD51 symbol:\n- should be updated to include pin types (input/output, etc)\n- should be divided into more (functional) units. \nRight now it is taking too much space
 Text Notes 8100 1300 0    50   Italic 0
-We might need to put the decoupling capacitors into the uC support block\nAlso, there are two more decoupling capacitors on sheet 1/3, so technically \ntwo mores capacitor are added to this list. Maybe we should remove the one \none sheet 1/3 and keep these ones below?
+We might need to put the decoupling capacitors into the uC support block
 Wire Notes Line
 	7250 4950 6050 4950

Commit message: Finished RF Connector
- Fixed alignment of schematic sheet 2
- Crated U.F connector symbol, layout, and 3D symbol
- Created coax symbol, layout, and 3D symbol
- Added RF connector to Schematic sheet 3
Other:
- moved on the sheet: C?, D?, J?, JP?, R?, U7, U?

Commit message: Fix: refactor symbol and modified schematics
Parts:
- removed C?: 100nF, symbol Device:CP1
- removed C? (x2): 15pF, symbol Device:C
- removed C?: 4.7uF, Capacitor_SMD:C_0603_1608Metric, symbol Device:C
- removed C? (x7): 100nF, Capacitor_SMD:C_0603_1608Metric, symbol Device:C
- removed IC?: SAMD51, Package_QFP:TQFP-100_14x14mm_P0.5mm, symbol Team-FIRE:SAMD51
- removed L?: 10uH, Inductor_SMD:L_0603_1608Metric, symbol Device:L
- removed R?: 10k, symbol Device:R
- removed R?: 330, symbol Device:R
- removed R?: 1k, symbol Device:R
- removed SW?: RESET, symbol Switch:SW_Push
- removed U?: ATSAMD51N20A-AU, QFP50P1600X1600X120-100N, symbol ATSAMD51N20A-AU-01:ATSAMD51N20A-AU
- removed Y?: 32.768kHz, symbol Device:Crystal
Connections:
- net labels removed: MISO, MOSI, SCK, SDA, SDL, SWO, XIN32, XOUT32
- wire segments 170 -> 83
Other:
- note removed: "A software reset is nice. But, we might need to\n manually reset the SAMD."
- note removed: "Crystal oscillator"
- note removed: "Pin 12"
- note removed: "Pin 39"
- note removed: "Pin 51"
- note removed: "Pin 63"
- note removed: "Pin 77"
- note removed: "Pin 89\n"
- note removed: "Pin 91\n"
- note removed: "Pin 92"
- note removed: "Place all components near\ntheir respective pins.\nChoose low ESR capacitors."
- note removed: "Reset button"
- note removed: "SAMD 51"
- note removed: "SWCLK Pin"
- note removed: "Should be closed to the SAMD \nto avoid crosstalk to other parts"
- note removed: "The SAMD51 symbol:\n- should be updated to include pin types (input/output, etc)\n- should be divided into more (functional) units. \nRight now it is taking too much space"
- note removed: "This shouldn't be block, just here as a note to add a pull-up resistor\nto ensure reliable operation"
- note removed: "We might need to put the decoupling capacitors into the uC support block"
- moved on the sheet: D?, J?, R?

Commit message: Fix connections
Parts:
- gave numbers to parts that had none: 9
Changed lines of the file:
@@
 	2650 3600 2100 3600
 $Comp
-L power:+3.3V #PWR?
+L power:+3.3V #PWR0139
 U 1 1 5E58E909
 P 2650 3500
-F 0 "#PWR?" H 2650 3350 50  0001 C CNN
+F 0 "#PWR0139" H 2650 3350 50  0001 C CNN
 F 1 "+3.3V" V 2750 3550 50  0000 C CNN
 F 2 "" H 2650 3500 50  0001 C CNN
@@
 $EndComp
 $Comp
-L power:GND #PWR?
+L power:GND #PWR0140
 U 1 1 5E57A4C5
 P 2100 3200
-F 0 "#PWR?" H 2100 2950 50  0001 C CNN
+F 0 "#PWR0140" H 2100 2950 50  0001 C CNN
 F 1 "GND" H 2350 3150 50  0000 R CNN
 F 2 "" H 2100 3200 50  0001 C CNN
@@
 $EndComp
 $Comp
-L Device:C C?
+L Device:C C19
 U 1 1 5E579B86
 P 2100 3350
-F 0 "C?" H 2000 3250 50  0000 C CNN
+F 0 "C19" H 2000 3250 50  0000 C CNN
 F 1 "0.1uF" H 1950 3450 50  0000 C CNN
 F 2 "Capacitor_SMD:C_0603_1608Metric" H 2138 3200 50  0001 C CNN
@@
 	3350 700  3350 5500
 $Comp
-L power:+5V #PWR?
+L power:+5V #PWR0141
 U 1 1 5E591E4C
 P 2650 3700
-F 0 "#PWR?" H 2650 3550 50  0001 C CNN
+F 0 "#PWR0141" H 2650 3550 50  0001 C CNN
 F 1 "+5V" V 2550 3750 50  0000 C CNN
 F 2 "" H 2650 3700 50  0001 C CNN
@@
 $EndComp
 $Comp
-L Connector_Generic:Conn_01x03 J?
+L Connector_Generic:Conn_01x03 J4
 U 1 1 5E58B8FE
 P 2850 3600
-F 0 "J?" V 2950 3650 50  0000 R CNN
+F 0 "J4" V 2950 3650 50  0000 R CNN
 F 1 "Conn_01x03" V 2950 3750 50  0001 R CNN
 F 2 "Connector_PinSocket_2.00mm:PinSocket_1x03_P2.00mm_Horizontal" H 2850 3600 50  0001 C CNN
@@
 $EndComp
 $Comp
-L power:+3.3V #PWR?
+L power:+3.3V #PWR0142
 U 1 1 5E561068
 P 1900 3500
-F 0 "#PWR?" H 1900 3350 50  0001 C CNN
+F 0 "#PWR0142" H 1900 3350 50  0001 C CNN
 F 1 "+3.3V" H 1850 3650 50  0000 C CNN
 F 2 "" H 1900 3500 50  0001 C CNN
@@
 	1600 4100 1400 4100
 $Comp
-L power:GND #PWR?
+L power:GND #PWR0143
 U 1 1 5E563F55
 P 1400 3600
-F 0 "#PWR?" H 1400 3350 50  0001 C CNN
+F 0 "#PWR0143" H 1400 3350 50  0001 C CNN
 F 1 "GND" V 1405 3472 50  0000 R CNN
 F 2 "" H 1400 3600 50  0001 C CNN
@@
 	1800 3600 1900 3600
 $Comp
-L Device:C C?
+L Device:C C18
 U 1 1 5E561EFE
 P 1650 3600
-F 0 "C?" V 1500 3500 50  0000 C CNN
+F 0 "C18" V 1500 3500 50  0000 C CNN
 F 1 "0.1uF" V 1600 3450 50  0000 C CNN
 F 2 "Capacitor_SMD:C_0603_1608Metric" H 1688 3450 50  0001 C CNN
@@
 	1900 3700 1900 3600
 $Comp
-L Device:R R?
+L Device:R R10
 U 1 1 5E55B090
 P 1500 5050
-F 0 "R?" H 1570 5096 50  0000 L CNN
+F 0 "R10" H 1570 5096 50  0000 L CNN
 F 1 "10k" H 1570 5005 50  0000 L CNN
 F 2 "Resistor_SMD:R_0603_1608Metric" V 1430 5050 50  0001 C CNN
@@
 $EndComp
 $Comp
-L power:GND #PWR?
+L power:GND #PWR0144
 U 1 1 5E554C34
 P 1500 5200
-F 0 "#PWR?" H 1500 4950 50  0001 C CNN
+F 0 "#PWR0144" H 1500 4950 50  0001 C CNN
 F 1 "GND" H 1505 5027 50  0000 C CNN
 F 2 "" H 1500 5200 50  0001 C CNN
@@
 	1600 3900 1500 3900
 $Comp
-L power:GND #PWR?
+L power:GND #PWR0145
 U 1 1 5E5500F4
 P 2000 5200
-F 0 "#PWR?" H 2000 4950 50  0001 C CNN
+F 0 "#PWR0145" H 2000 4950 50  0001 C CNN
 F 1 "GND" H 2005 5027 50  0000 C CNN
 F 2 "" H 2000 5200 50  0001 C CNN
@@
 	1700 1000 1700 1100
 $Comp
-L power:+3.3V #PWR?
+L power:+3.3V #PWR0146
 U 1 1 5E50DD7A
 P 1700 1000
-F 0 "#PWR?" H 1700 850 50  0001 C CNN
+F 0 "#PWR0146" H 1700 850 50  0001 C CNN
 F 1 "+3.3V" H 1700 1150 50  0000 C CNN
 F 2 "" H 1700 1000 50  0001 C CNN
@@
 $EndComp
 $Comp
-L Jumper:SolderJumper_3_Bridged12 JP?
+L Jumper:SolderJumper_3_Bridged12 JP2
 U 1 1 5E50B8B0
 P 1400 1100
-F 0 "JP?" H 1400 1213 50  0000 C CNN
+F 0 "JP2" H 1400 1213 50  0000 C CNN
 F 1 "SolderJumper_3_Bridged12" H 1400 1214 50  0001 C CNN
 F 2 "" H 1400 1100 50  0001 C CNN
@@
 	1400 1350 1400 1250
 $Comp
-L power:GND #PWR?
+L power:GND #PWR0147
 U 1 1 5E50A8F7
 P 1400 1450
-F 0 "#PWR?" H 1400 1200 50  0001 C CNN
+F 0 "#PWR0147" H 1400 1200 50  0001 C CNN
 F 1 "GND" H 1405 1277 50  0000 C CNN
 F 2 "" H 1400 1450 50  0001 C CNN
@@
 	2500 1350 2600 1350
 $Comp
-L Device:C C?
+L Device:C C17
 U 1 1 5E508BEB
 P 1650 1350
-F 0 "C?" V 1500 1450 50  0000 C CNN
+F 0 "C17" V 1500 1450 50  0000 C CNN
 F 1 "0.1uF" V 1600 1500 50  0000 C CNN
 F 2 "Capacitor_SMD:C_0603_1608Metric" H 1688 1200 50  0001 C CNN
@@
 EN_IR_BUS
 $Comp
-L power:GND #PWR?
+L power:GND #PWR0148
 U 1 1 5E5076A4
 P 1500 2950
-F 0 "#PWR?" H 1500 2700 50  0001 C CNN
+F 0 "#PWR0148" H 1500 2700 50  0001 C CNN
 F 1 "GND" H 1350 2900 50  0000 C CNN
 F 2 "" H 1500 2950 50  0001 C CNN
@@
 $EndComp
 $Comp
-L Device:R R?
+L Device:R R9
 U 1 1 5E5071DF
 P 1500 2800
-F 0 "R?" H 1570 2846 50  0000 L CNN
+F 0 "R9" H 1570 2846 50  0000 L CNN
 F 1 "10k" H 1570 2755 50  0000 L CNN
 F 2 "Resistor_SMD:R_0603_1608Metric" V 1430 2800 50  0001 C CNN
@@
 	1400 1850 1600 1850
 $Comp
-L Device:C C?
+L Device:C C20
 U 1 1 5E502C68
 P 2350 1350
-F 0 "C?" V 2200 1450 50  0000 C CNN
+F 0 "C20" V 2200 1450 50  0000 C CNN
 F 1 "0.1uF" V 2300 1500 50  0000 C CNN
 F 2 "Capacitor_SMD:C_0603_1608Metric" H 2388 1200 50  0001 C CNN
@@
 $EndComp
 $Comp
-L power:GND #PWR?
+L power:GND #PWR0149
 U 1 1 5E503AC6
 P 2600 1350
-F 0 "#PWR?" H 2600 1100 50  0001 C CNN
+F 0 "#PWR0149" H 2600 1100 50  0001 C CNN
 F 1 "GND" V 2605 1222 50  0000 R CNN
 F 2 "" H 2600 1350 50  0001 C CNN
@@
 	2100 1250 2100 1350
 $Comp
-L Logic_LevelTranslator:TXB0108DQSR U?
+L Logic_LevelTranslator:TXB0108DQSR U4
 U 1 1 5E4FCEC1
 P 2000 2150
-F 0 "U?" H 2150 1450 50  0000 C CNN
+F 0 "U4" H 2150 1450 50  0000 C CNN
 F 1 "TXB0108DQSR" H 2350 1350 50  0000 C CNN
 F 2 "Package_SON:USON-20_2x4mm_P0.4mm" H 2000 1400 50  0001 C CNN
@@
 $EndComp
 $Comp
-L power:+3.3V #PWR?
+L power:+3.3V #PWR0150
 U 1 1 5E500FDB
 P 2100 1250
-F 0 "#PWR?" H 2100 1100 50  0001 C CNN
+F 0 "#PWR0150" H 2100 1100 50  0001 C CNN
 F 1 "+3.3V" H 2100 1400 50  0000 C CNN
 F 2 "" H 2100 1250 50  0001 C CNN
@@
 IO-DTR
 $Comp
-L power:GND #PWR?
+L power:GND #PWR0151
 U 1 1 5E4FE4B4
 P 2000 2950
-F 0 "#PWR?" H 2000 2700 50  0001 C CNN
+F 0 "#PWR0151" H 2000 2700 50  0001 C CNN
 F 1 "GND" H 1850 2900 50  0000 C CNN
 F 2 "" H 2000 2950 50  0001 C CNN
