File: Board Redesign/KiCad Project/Team-FIRE-v2/schematic-1.sch (KiCad schematic (older format))
At the start: 32 parts

Commit message: Fix connections
Parts:
- gave numbers to parts that had none: 32
